Commit message: placed 3 frankas urdf in a (60,60,60) triangle around x,y= 0,0

File: curobo/src/curobo/content/assets/robot/franka_3_arm/franka_3_arm.urdf (robot description, URDF)
Before this commit: robot franka_3_arm, 43 links, 42 joints
Joints:
- joint arm_0_arm_fixed: origin xyz=-1.0 0.0 0.0 rpy=0 0 0 -> xyz=-0.7071 -0.5 0.0 rpy=0 0 0
- joint arm_1_arm_fixed: origin xyz=0.0 0.0 0.0 rpy=0 0 0 -> xyz=0.7071 -0.5 0.0 rpy=0 0 0
- joint arm_2_arm_fixed: origin xyz=1.0 0.0 0.0 rpy=0 0 0 -> xyz=0.0 0.5 0.0 rpy=0 0 0
