Commit message: 4 arm example of frankas (centralized planning) ready at:

File: curobo/src/curobo/content/assets/robot/franka_4_arm/franka_4_arm.urdf (robot description, URDF)
Before this commit: robot franka_4_arm, 57 links, 56 joints
Joints:
- joint arm_0_arm_fixed: origin xyz=-1.5 0.0 0.0 rpy=0 0 0 -> xyz=-0.5 -0.5 0.0 rpy=0 0 0
- joint arm_1_arm_fixed: origin xyz=-0.5 0.0 0.0 rpy=0 0 0 -> xyz=-0.5 0.5 0.0 rpy=0 0 0
- joint arm_2_arm_fixed: origin xyz=0.5 0.0 0.0 rpy=0 0 0 -> xyz=0.5 0.5 0.0 rpy=0 0 0
- joint arm_3_arm_fixed: origin xyz=1.5 0.0 0.0 rpy=0 0 0 -> xyz=0.5 -0.5 0.0 rpy=0 0 0
