Commit message: wip g1: bugfixing, now solved the rollouts visualization. TBD: sphere visualization, solve bound cost issue (enters 'recovery mode')

File: curobo/src/curobo/content/assets/robot/g1_humanoid/f.urdf (robot description, URDF)
Before this commit: robot g1, 44 links, 43 joints
Links:
- removed link g1
- added link pelvis; visual mesh filename=urdf_mesh/pelvis_visuals.obj scale=1. 1. 1.
Joints:
- joint left_hip_pitch_joint: parent g1 -> pelvis
- joint pelvis_contour_joint: parent g1 -> pelvis
- joint right_hip_pitch_joint: parent g1 -> pelvis
- joint torso_joint: parent g1 -> pelvis
