Commit message: single mpc based on wmv for general usage

File: curobo/src/curobo/content/assets/robot/g1_23dof_description/g1_23dofs_cfgs/g1_23dof_original.urdf (robot description, URDF)
Before this commit: robot g1_23dof, 34 links, 33 joints
Links:
- removed link dummy_ee_left_link
Joints:
- removed joint dummy_ee_left_joint
