Commit message: wip

File: curobo/src/curobo/content/assets/robot/simple_disk_description/simple_disk.urdf (robot description, URDF)
Before this commit: robot simple_disk, 4 links, 3 joints
Links:
- removed link base_link_x
- removed link base_link_y
- removed link disk_base
- added link ee_link, mass 0.001
- added link mobile_base, mass 0.001
- added link world, mass 0.001
- link base_link: mass 0.001 -> 2.0; geometry collision cylinder length=0.1 radius=0.15; visual cylinder length=0.1 radius=0.15
Joints:
- removed joint base_theta
- added joint base_to_ee: type fixed, parent base_link, child ee_link, origin xyz=0 0 0.0 rpy=0 0 0.0
- joint base_x: child base_link_x -> mobile_base; parent base_link -> world
- joint base_y: child base_link_y -> base_link; parent base_link_x -> mobile_base

Commit message: wip

File: curobo/src/curobo/content/assets/robot/simple_disk_description/simple_disk.urdf (robot description, URDF)
Before this commit: robot simple_disk, 4 links, 3 joints
Links:
- removed link mobile_base
- added link intermediate, mass 0.001
- link base_link: geometry collision cylinder length=0.1 radius=0.1; visual cylinder length=0.1 radius=0.1
Joints:
- removed joint base_x
- removed joint base_y
- added joint joint_x: type prismatic, parent world, child intermediate, origin xyz=0 0 0 rpy=0 0 0, axis 1 0 0, limit lower=-100 upper=100 effort=10 velocity=0.5
- added joint joint_y: type prismatic, parent intermediate, child base_link, origin xyz=0 0 0 rpy=0 0 0, axis 0 1 0, limit lower=-100 upper=100 effort=10 velocity=0.5
- joint base_to_ee: origin xyz=0 0 0.0 rpy=0 0 0.0 -> xyz=0 0 0 rpy=0 0 0
