Commit message: wip

File: curobo/src/curobo/content/assets/robot/simple_disk_description/simple_disk_tiny.urdf (robot description, URDF)
Before this commit: robot simple_disk, 4 links, 3 joints
Links:
- link base_link: mass 2.0 -> 0.5; geometry collision cylinder length=0.01 radius=0.025; visual cylinder length=0.02 radius=0.025
Joints:
- joint joint_x: limit lower=-100 upper=100 effort=10 velocity=2.0 -> lower=-100 upper=100 effort=1 velocity=1.0
- joint joint_y: limit lower=-100 upper=100 effort=10 velocity=2.0 -> lower=-100 upper=100 effort=1 velocity=1.0

Commit message: wip

File: curobo/src/curobo/content/assets/robot/simple_disk_description/simple_disk_tiny.urdf (robot description, URDF)
Before this commit: robot simple_disk, 4 links, 3 joints
Joints:
- joint joint_x: limit lower=-100 upper=100 effort=1 velocity=1.0 -> lower=-100 upper=100 effort=10 velocity=2.0
- joint joint_y: limit lower=-100 upper=100 effort=1 velocity=1.0 -> lower=-100 upper=100 effort=10 velocity=2.0

Commit message: wip

File: curobo/src/curobo/content/assets/robot/simple_disk_description/simple_disk_tiny.urdf (robot description, URDF)
Before this commit: robot simple_disk, 4 links, 3 joints
Links:
- link base_link: mass 0.5 -> 0.01
Joints:
- joint joint_x: limit lower=-100 upper=100 effort=10 velocity=2.0 -> lower=-100 upper=100 effort=100 velocity=2.0
- joint joint_y: limit lower=-100 upper=100 effort=10 velocity=2.0 -> lower=-100 upper=100 effort=100 velocity=2.0

Commit message: current cost config looks fine in 4 disk robots with wall

File: curobo/src/curobo/content/assets/robot/simple_disk_description/simple_disk_tiny.urdf (robot description, URDF)
Before this commit: robot simple_disk, 4 links, 3 joints
Links:
- link base_link: mass 0.01 -> 0.1
Joints:
- joint joint_x: limit lower=-100 upper=100 effort=100 velocity=2.0 -> lower=-100 upper=100 effort=1000 velocity=5.0
- joint joint_y: limit lower=-100 upper=100 effort=100 velocity=2.0 -> lower=-100 upper=100 effort=1000 velocity=5.0

Commit message: wip: experimental change-cost func to minimal distance based (relu like)

File: curobo/src/curobo/content/assets/robot/simple_disk_description/simple_disk_tiny.urdf (robot description, URDF)
Before this commit: robot simple_disk, 4 links, 3 joints
Joints:
- joint joint_x: limit lower=-100 upper=100 effort=1000 velocity=5.0 -> lower=-100 upper=100 effort=100 velocity=3.0
- joint joint_y: limit lower=-100 upper=100 effort=1000 velocity=5.0 -> lower=-100 upper=100 effort=100 velocity=3.0

Commit message: wip-before merging dynamic obs new

File: curobo/src/curobo/content/assets/robot/simple_disk_description/simple_disk_tiny.urdf (robot description, URDF)
Before this commit: robot simple_disk, 4 links, 3 joints
Joints:
- joint joint_x: limit lower=-100 upper=100 effort=100 velocity=3.0 -> lower=-100 upper=100 effort=10 velocity=0.35
- joint joint_y: limit lower=-100 upper=100 effort=100 velocity=3.0 -> lower=-100 upper=100 effort=10 velocity=0.35

Commit message: disk changes. Commit before mergeing bugfix from remote

File: curobo/src/curobo/content/assets/robot/simple_disk_description/simple_disk_tiny.urdf (robot description, URDF)
Before this commit: robot simple_disk, 4 links, 3 joints
Joints:
- joint joint_x: limit lower=-100 upper=100 effort=10 velocity=0.35 -> lower=-5.0 upper=5.0 effort=87 velocity=1.0
- joint joint_y: limit lower=-100 upper=100 effort=10 velocity=0.35 -> lower=-5.0 upper=5.0 effort=87 velocity=1.0
