Commit message: ur5e dual

File: curobo/src/curobo/content/assets/robot/ur_description/dual_ur5e_05.urdf (robot description, URDF)
Before this commit: robot ur5e_robot, 41 links, 40 joints
Links:
- removed link base_link_2
- removed link base_link_3
- removed link base_link_inertia_link_2
- removed link base_link_inertia_link_3
- removed link flange_2
- removed link flange_3
- removed link forearm_link_2
- removed link forearm_link_3
- removed link shoulder_link_2
- removed link shoulder_link_3
- removed link tool2
- removed link tool3
- removed link upper_arm_link_2
- removed link upper_arm_link_3
- removed link wrist_1_link_2
- removed link wrist_1_link_3
- removed link wrist_2_link_2
- removed link wrist_2_link_3
- removed link wrist_3_link_2
- removed link wrist_3_link_3
Joints:
- removed joint base_fixture_j_base_link_2
- removed joint base_fixture_j_base_link_3
- removed joint base_link_base_link_inertia_joint_2
- removed joint base_link_base_link_inertia_joint_3
- removed joint elbow_joint_2
- removed joint elbow_joint_3
- removed joint flange_tool_joint_2
- removed joint flange_tool_joint_3
- removed joint shoulder_lift_joint_2
- removed joint shoulder_lift_joint_3
- removed joint shoulder_pan_joint_2
- removed joint shoulder_pan_joint_3
- removed joint wrist_1_joint_2
- removed joint wrist_1_joint_3
- removed joint wrist_2_joint_2
- removed joint wrist_2_joint_3
- removed joint wrist_3_flange_joint_2
- removed joint wrist_3_flange_joint_3
- removed joint wrist_3_joint_2
- removed joint wrist_3_joint_3
