Commit message: rotated quad_ur5e_04

File: curobo/src/curobo/content/assets/robot/ur_description/quad_ur5e_04.urdf (robot description, URDF)
Before this commit: robot ur5e_robot, 41 links, 40 joints
Joints:
- joint base_fixture_j_base_link: origin xyz=0.4 0.4 0 rpy=0 0 0 -> xyz=0.4 0.4 0 rpy=0 0 2.355
- joint base_fixture_j_base_link_1: origin xyz=-0.4 0.4 0 rpy=0 0 0.0 -> xyz=-0.4 0.4 0 rpy=0 0 0.785
- joint base_fixture_j_base_link_2: origin xyz=0.4 -0.4 0 rpy=0 0 3.14 -> xyz=0.4 -0.4 0 rpy=0 0 3.925
- joint base_fixture_j_base_link_3: origin xyz=-0.4 -0.4 0 rpy=0 0 3.14 -> xyz=-0.4 -0.4 0 rpy=0 0 5.495
