Commit message: improved self penetration awareness (robot avoids passsing its arm from within its body)

File: curobo/src/curobo/content/assets/robot/g1_feb26/unitreerobotics unitree_ros master robots-g1_description/g1_left_arm.urdf (robot description, URDF)
Before this commit: robot g1_left_arm, 19 links, 18 joints
Links:
- link waist_roll_link: geometry collision mesh filename=meshes/waist_roll_link.STL; visual mesh filename=meshes/waist_roll_link.STL
- link waist_yaw_link: geometry collision mesh filename=meshes/waist_yaw_link.STL; visual mesh filename=meshes/waist_yaw_link.STL
