Commit message: improved left arm only

File: curobo/src/curobo/content/assets/robot/g1_feb26/unitreerobotics unitree_ros master robots-g1_description/g1_left_arm_only.urdf (robot description, URDF)
Before this commit: robot g1_left_arm_only, 10 links, 9 joints
Joints:
- joint left_shoulder_pitch_joint: origin xyz=0.0039563 0.10022 0.23778 rpy=0.27931 5.4949E-05 -0.00019159 -> xyz=-0.0000072 0.10022 0.29178 rpy=0.27931 5.4949E-05 -0.00019159

Commit message: changed ee to be on middle finger tip in both arms

File: curobo/src/curobo/content/assets/robot/g1_feb26/unitreerobotics unitree_ros master robots-g1_description/g1_left_arm_only.urdf (robot description, URDF)
Before this commit: robot g1_left_arm_only, 10 links, 9 joints
Joints:
- joint dummy_ee_left_joint: origin xyz=0.1 0 0 rpy=0 0 0 -> xyz=0.13 -0.05 -0.001 rpy=0 0 0

File: curobo/src/curobo/content/assets/robot/g1_feb26/unitreerobotics unitree_ros master robots-g1_description/g1_right_arm_only.urdf (robot description, URDF)
Before this commit: robot g1_right_arm_only, 10 links, 9 joints
Joints:
- joint dummy_ee_right_joint: origin xyz=0.1 0 0 rpy=0 0 0 -> xyz=0.13 0.05 0 rpy=0 0 0

Commit message: wip

File: curobo/src/curobo/content/assets/robot/g1_feb26/unitreerobotics unitree_ros master robots-g1_description/g1_left_arm_only.urdf (robot description, URDF)
Before this commit: robot g1_left_arm_only, 10 links, 9 joints
Joints:
- joint left_wrist_yaw_joint: limit lower=-1.614429558 upper=1.614429558 effort=5 velocity=22 -> lower=-1.0 upper=1.0 effort=5 velocity=22

File: curobo/src/curobo/content/assets/robot/g1_feb26/unitreerobotics unitree_ros master robots-g1_description/g1_right_arm_only.urdf (robot description, URDF)
Before this commit: robot g1_right_arm_only, 10 links, 9 joints
Joints:
- joint right_wrist_yaw_joint: limit lower=-1.614429558 upper=1.614429558 effort=5 velocity=22 -> lower=-1.0 upper=1.0 effort=5 velocity=22
